Commit message: added more features
added camera plugin

File: my_robot/my_urdfs/cam_model.urdf.xacro (robot description, xacro)
@@ -15,4 +15,5 @@
 <xacro:property name="rod_radius" value='0.018' />
 <xacro:property name="rod_length" value='0.3'/>
+<xacro:property name="camera_dim" value="0.01"/>
 <material name="blue">
     <color rgba="0.1 0.0 0.9 1"/>
@@ -121,5 +122,5 @@
       </actuator>
       <joint name="${prefix}_${suffix}_scylinder_wheel">
-        <hardwareInterface>VelocityJointInterface</hardwareInterface>
+        <hardwareInterface>hardware_interface/VelocityJointInterface</hardwareInterface>
       </joint>
     </transmission>
@@ -175,11 +176,33 @@
 <transmission name="cylin_trans">
     <type>transmission_interface/SimpleTransmission</type>
-    <actuator name="$cylin_motor">
+    <actuator name="motor1">
       <mechanicalReduction>1</mechanicalReduction>
     </actuator>
     <joint name="rod_cylin">
-      <hardwareInterface>PositionJointInterface</hardwareInterface>
+      <hardwareInterface>hardware_interface/PositionJointInterface</hardwareInterface>
     </joint>
 </transmission>
+<link name="camera_link">
+    <visual>
+        <geometry>
+            <box size="${camera_dim} ${camera_dim} ${camera_dim}"/>
+        </geometry>
+    </visual>
+    <collision>
+        <geometry>
+            <box size="${camera_dim} ${camera_dim} ${camera_dim}"/>
+        </geometry>
+    </collision>
+    <inertial>
+        <mass value="0.2"/>
+       <inertia ixx="0.0000033333" ixy="0.0" ixz="0.0" iyy="0.0000033333" iyz="0.0" izz="0.0000033333"/>
+    </inertial>
+</link>
+<joint name="camera_joint" type="fixed">
+    <axis xyz="1.0 0.0 0.0"/>
+    <parent link="cylin"/>
+    <child link="camera_link"/>
+    <origin xyz="0.075 0.0 0.02"/>
+</joint>
 <gazebo>
     <plugin name="gazebo_ros_control" filename="libgazebo_ros_control.so">
@@ -187,3 +210,42 @@
     </plugin>
 </gazebo>
+<gazebo reference="camera_link">
+    <sensor type="camera" name="camera1">
+      <update_rate>30.0</update_rate>
+      <camera name="head">
+        <horizontal_fov>1.3962634</horizontal_fov>
+        <image>
+          <width>800</width>
+          <height>800</height>
+          <format>R8G8B8</format>
+        </image>
+        <!-- <save enabled='true'>
+            <path>/home/fierce/turtlebot_photos</path>
+        </save> -->
+        <clip>
+          <near>0.02</near>
+          <far>300</far>
+        </clip>
+        <noise>
+          <type>gaussian</type>
+          <mean>0.0</mean>
+          <stddev>0.007</stddev>
+        </noise>
+      </camera>
+      <plugin name="camera_controller" filename="libgazebo_ros_camera.so">
+        <alwaysOn>true</alwaysOn>
+        <updateRate>0.0</updateRate>
+        <cameraName>macroed/camera1</cameraName>
+        <imageTopicName>image_raw</imageTopicName>
+        <cameraInfoTopicName>camera_info</cameraInfoTopicName>
+        <frameName>camera_link</frameName>
+        <hackBaseline>0.07</hackBaseline>
+        <distortionK1>0.0</distortionK1>
+        <distortionK2>0.0</distortionK2>
+        <distortionK3>0.0</distortionK3>
+        <distortionT1>0.0</distortionT1>
+        <distortionT2>0.0</distortionT2>
+      </plugin>
+    </sensor>
+  </gazebo>
 </robot>

Commit message: Added lasers

File: my_robot/my_urdfs/cam_model.urdf.xacro (robot description, xacro)
@@ -16,4 +16,7 @@
 <xacro:property name="rod_length" value='0.3'/>
 <xacro:property name="camera_dim" value="0.01"/>
+<xacro:property name="pi" value="3.1428"/>
+<xacro:property name="laz_radius" value="0.04"/>
+<xacro:property name="laz_height" value="0.1"/>
 <material name="blue">
     <color rgba="0.1 0.0 0.9 1"/>
@@ -249,3 +252,9 @@
     </sensor>
   </gazebo>
+<xacro:include filename="$(find my_robot)/my_urdfs/lidar.urdf.xacro"/>
+  <joint name="lidarGlue" type="fixed">
+    <parent link="base_link"/>
+    <child link="laz_base"/>
+    <origin xyz="${width/4} 0 ${height/2}"/>
+  </joint>
 </robot>

Commit message: Commit1

File: my_robot/my_urdfs/cam_model.urdf.xacro (robot description, xacro)
@@ -110,5 +110,5 @@
         <parent link="${prefix}_${suffix}_scylinder"/>
         <child link="${prefix}_${suffix}_wheel"/>
-        <origin xyz="0.0 0.0 -0.07" rpy="1.57 0.0 0.0"/>
+        <origin xyz="0.0 0.0 -0.07" rpy="-1.57 0.0 0.0"/>
     </joint>
     <gazebo reference="${prefix}_${suffix}_wheel">
@@ -252,9 +252,70 @@
     </sensor>
   </gazebo>
-<xacro:include filename="$(find my_robot)/my_urdfs/lidar.urdf.xacro"/>
+<!-- <xacro:include filename="$(find my_robot)/my_urdfs/lidar.urdf.xacro"/>
   <joint name="lidarGlue" type="fixed">
     <parent link="base_link"/>
     <child link="laz_base"/>
     <origin xyz="${width/4} 0 ${height/2}"/>
+  </joint> -->
+  <joint name="hokuyo_joint" type="fixed">
+    <axis xyz="0 0 1" />
+    <origin xyz="0.12 0 0.13" rpy="0 0 0"/>
+    <parent link="base_link"/>
+    <child link="hokuyo_link"/>
   </joint>
+  <!-- Hokuyo Laser -->
+  <link name="hokuyo_link">
+    <collision>
+      <origin xyz="0 0 0" rpy="0 0 0"/>
+      <geometry>
+    <box size="0.1 0.1 0.1"/>
+      </geometry>
+    </collision>
+    <visual>
+      <origin xyz="0 0 0" rpy="0 0 0"/>
+      <geometry>
+        <box size="0.1 0.1 0.1"/>
+      </geometry>
+    </visual>
+    <inertial>
+      <mass value="1e-5" />
+      <origin xyz="0 0 0" rpy="0 0 0"/>
+      <inertia ixx="1e-6" ixy="0" ixz="0" iyy="1e-6" iyz="0" izz="1e-6" />
+    </inertial>
+  </link>
+  <gazebo reference="hokuyo_link">
+    <sensor type="gpu_ray" name="head_hokuyo_sensor">
+      <pose>0 0 0 0 0 0</pose>
+      <visualize>true</visualize>
+      <update_rate>40</update_rate>
+      <ray>
+        <scan>
+          <horizontal>
+            <samples>720</samples>
+            <resolution>1</resolution>
+            <min_angle>-1.570796</min_angle>
+            <max_angle>1.570796</max_angle>
+          </horizontal>
+        </scan>
+        <range>
+          <min>0.10</min>
+          <max>10.0</max>
+          <resolution>0.01</resolution>
+        </range>
+        <noise>
+          <type>gaussian</type>
+          <!-- Noise parameters based on published spec for Hokuyo laser
+               achieving "+-30mm" accuracy at range < 10m.  A mean of 0.0m and
+               stddev of 0.01m will put 99.7% of samples within 0.03m of the true
+               reading. -->
+          <mean>0.05</mean>
+          <stddev>0.01</stddev>
+        </noise>
+      </ray>
+      <plugin name="gazebo_ros_head_hokuyo_controller" filename="libgazebo_ros_gpu_laser.so">
+        <topicName>/macroed/laser/scan</topicName>
+        <frameName>hokuyo_link</frameName>
+      </plugin>
+    </sensor>
+  </gazebo>
 </robot>
